Commit message: Tune B002 3D scene object positions

File: generated/room_furniture_3d.urdf (robot description, URDF)
Before this commit: robot room_furniture, 97 links, 96 joints
Joints:
- joint furn_43_j: origin xyz=0.4200 3.5000 1.1200 rpy=0 0 0 -> xyz=-0.1000 4.2000 1.1200 rpy=0 0 0
- joint furn_44_j: origin xyz=0.4200 3.5000 0.8400 rpy=0 0 0 -> xyz=-0.1000 4.2000 0.8400 rpy=0 0 0
- joint furn_45_j: origin xyz=0.4200 3.5000 0.0400 rpy=0 0 0 -> xyz=-0.1000 4.2000 0.0400 rpy=0 0 0
- joint furn_46_j: origin xyz=0.6000 3.5000 0.3200 rpy=0 1.5708 0 -> xyz=-0.3000 3.4800 0.3200 rpy=0 1.5708 0
- joint furn_47_j: origin xyz=0.3000 3.5000 0.5800 rpy=0 0 0 -> xyz=-0.4200 3.4800 0.5800 rpy=0 0 0
